File: training_hardware/training_hardware.kicad_sch (KiCad schematic)
At the start: 0 parts

Commit message: add can
Other:
- added sheet CAN (CAN.kicad_sch)
Changed lines of the file:
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@@
 	(paper "A4")
+	(sheet
+		(at 34.29 96.52)
+		(size 55.88 43.18)
+		(exclude_from_sim no)
+		(in_bom yes)
+		(on_board yes)
+		(dnp no)
+		(fields_autoplaced yes)
+		(stroke
+			(width 0.1524)
+			(type solid)
+		)
+		(fill
+			(color 0 0 0 0.0000)
+		)
+		(property "Sheetname" "CAN"
+			(at 34.29 95.8084 0)
+			(effects
+				(font
+					(size 1.27 1.27)
+				)
+				(justify left bottom)
+			)
+		)
+		(property "Sheetfile" "CAN.kicad_sch"
+			(at 34.29 140.2846 0)
+			(effects
+				(font
+					(size 1.27 1.27)
+				)
+				(justify left top)
+			)
+		)
+		(instances
+			(project "training_hardware"
+				(path "/ce6aff0a-6a24-4161-b195-5f43ae1bbb8d"
+					(page "4")
+				)
+			)
+		)
+	)
 	(sheet
 		(at 180.34 91.44)

Commit message: finish schematic
Other:
- sheet CAN ports: added RXD, STBY, TXD; removed none
- sheet MCU ports: added CRX1, CTX1, STBY; removed none
Changed lines of the file:
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@@
 	(generator_version "9.0")
 	(paper "A4")
+	(wire
+		(pts
+			(xy 76.2 110.49) (xy 101.6 110.49)
+		)
+		(stroke
+			(width 0)
+			(type default)
+		)
+	)
+	(wire
+		(pts
+			(xy 76.2 118.11) (xy 101.6 118.11)
+		)
+		(stroke
+			(width 0)
+			(type default)
+		)
+	)
+	(wire
+		(pts
+			(xy 76.2 114.3) (xy 101.6 114.3)
+		)
+		(stroke
+			(width 0)
+			(type default)
+		)
+	)
 	(sheet
-		(at 34.29 96.52)
-		(size 55.88 43.18)
+		(at 25.4 101.6)
+		(size 50.8 25.4)
 		(exclude_from_sim no)
 		(in_bom yes)
@@
 		)
 		(property "Sheetname" "CAN"
-			(at 34.29 95.8084 0)
+			(at 25.4 100.8884 0)
 			(effects
 				(font
@@
 		)
 		(property "Sheetfile" "CAN.kicad_sch"
-			(at 34.29 140.2846 0)
+			(at 25.4 127.5846 0)
 			(effects
 				(font
@@
 				)
 				(justify left top)
+			)
+		)
+		(pin "RXD" output
+			(at 76.2 110.49 0)
+			(effects
+				(font
+					(size 1.27 1.27)
+				)
+				(justify right)
+			)
+		)
+		(pin "STBY" input
+			(at 76.2 114.3 0)
+			(effects
+				(font
+					(size 1.27 1.27)
+				)
+				(justify right)
+			)
+		)
+		(pin "TXD" input
+			(at 76.2 118.11 0)
+			(effects
+				(font
+					(size 1.27 1.27)
+				)
+				(justify right)
 			)
 		)
@@
 	)
 	(sheet
-		(at 180.34 91.44)
-		(size 55.88 48.26)
+		(at 177.8 101.6)
+		(size 50.8 25.4)
 		(exclude_from_sim no)
 		(in_bom yes)
@@
 		)
 		(property "Sheetname" "Power"
-			(at 180.34 90.7284 0)
+			(at 177.8 100.8884 0)
 			(effects
 				(font
@@
 		)
 		(property "Sheetfile" "power.kicad_sch"
-			(at 180.34 140.2846 0)
+			(at 177.8 127.5846 0)
 			(effects
 				(font
@@
 	)
 	(sheet
-		(at 102.87 92.71)
-		(size 57.15 45.72)
+		(at 101.6 101.6)
+		(size 50.8 25.4)
 		(exclude_from_sim no)
 		(in_bom yes)
@@
 		)
 		(property "Sheetname" "MCU"
-			(at 102.87 91.9984 0)
+			(at 101.6 100.8884 0)
 			(effects
 				(font
@@
 		)
 		(property "Sheetfile" "MCU.kicad_sch"
-			(at 102.87 139.0146 0)
+			(at 101.6 127.5846 0)
 			(effects
 				(font
@@
 			)
 		)
+		(pin "CRX1" input
+			(at 101.6 110.49 180)
+			(effects
+				(font
+					(size 1.27 1.27)
+				)
+				(justify left)
+			)
+		)
+		(pin "CTX1" output
+			(at 101.6 118.11 180)
+			(effects
+				(font
+					(size 1.27 1.27)
+				)
+				(justify left)
+			)
+		)
+		(pin "STBY" output
+			(at 101.6 114.3 180)
+			(effects
+				(font
+					(size 1.27 1.27)
+				)
+				(justify left)
+			)
+		)
