File: Training_Hardware/Training_Hardware.kicad_sch (KiCad schematic)
At the start: 0 parts

Commit message: Add CAN Transmitter
Other:
- added sheet CAN (CAN.kicad_sch)
Changed lines of the file:
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@@
+	)
+	(sheet
+		(at 99.06 83.82)
+		(size 27.94 12.7)
+		(exclude_from_sim no)
+		(in_bom yes)
+		(on_board yes)
+		(dnp no)
+		(fields_autoplaced yes)
+		(stroke
+			(width 0.1524)
+			(type solid)
+		)
+		(fill
+			(color 0 0 0 0.0000)
+		)
+		(property "Sheetname" "CAN"
+			(at 99.06 83.1084 0)
+			(effects
+				(font
+					(size 1.27 1.27)
+				)
+				(justify left bottom)
+			)
+		)
+		(property "Sheetfile" "CAN.kicad_sch"
+			(at 99.06 97.1046 0)
+			(effects
+				(font
+					(size 1.27 1.27)
+				)
+				(justify left top)
+			)
+		)
+		(instances
+			(project "Training_Hardware"
+				(path "/b0d5b3f6-1860-46b8-b850-3c3e521e5123"
+					(page "4")
+				)
+			)
+		)
 	)
 	(sheet

Commit message: Finish Schematic
Other:
- sheet CAN ports: added RXD, STBY, TXD; removed none
- sheet MCU ports: added CRX 1, CTX 1, STBY; removed none
Changed lines of the file:
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@@
 	(generator_version "9.0")
 	(paper "A4")
+	(wire
+		(pts
+			(xy 127 92.71) (xy 135.89 92.71)
+		)
+		(stroke
+			(width 0)
+			(type default)
+		)
+	)
+	(wire
+		(pts
+			(xy 127 87.63) (xy 135.89 87.63)
+		)
+		(stroke
+			(width 0)
+			(type default)
+		)
+	)
+	(wire
+		(pts
+			(xy 127 90.17) (xy 135.89 90.17)
+		)
+		(stroke
+			(width 0)
+			(type default)
+		)
+	)
 	(sheet
-		(at 135.89 67.31)
+		(at 120.65 63.5)
 		(size 22.86 11.43)
 		(exclude_from_sim no)
@@
 		)
 		(property "Sheetname" "Power"
-			(at 135.89 66.5984 0)
+			(at 120.65 62.7884 0)
 			(effects
 				(font
@@
 		)
 		(property "Sheetfile" "Power.kicad_sch"
-			(at 135.89 79.3246 0)
+			(at 120.65 75.5146 0)
 			(effects
 				(font
@@
 			)
 		)
+		(pin "RXD" output
+			(at 127 87.63 0)
+			(effects
+				(font
+					(size 1.27 1.27)
+				)
+				(justify right)
+			)
+		)
+		(pin "STBY" input
+			(at 127 90.17 0)
+			(effects
+				(font
+					(size 1.27 1.27)
+				)
+				(justify right)
+			)
+		)
+		(pin "TXD" input
+			(at 127 92.71 0)
+			(effects
+				(font
+					(size 1.27 1.27)
+				)
+				(justify right)
+			)
+		)
 		(instances
 			(project "Training_Hardware"
@@
 	)
 	(sheet
-		(at 135.89 99.06)
-		(size 22.86 10.16)
+		(at 135.89 83.82)
+		(size 31.75 12.7)
 		(exclude_from_sim no)
 		(in_bom yes)
@@
 		)
 		(property "Sheetname" "MCU"
-			(at 136.144 98.806 0)
+			(at 136.144 83.566 0)
 			(effects
 				(font
@@
 		)
 		(property "Sheetfile" "MCU.kicad_sch"
-			(at 135.89 109.8046 0)
+			(at 135.89 97.282 0)
 			(effects
 				(font
@@
 			)
 		)
+		(pin "CRX 1" input
+			(at 135.89 87.63 180)
+			(effects
+				(font
+					(size 1.27 1.27)
+				)
+				(justify left)
+			)
+		)
+		(pin "CTX 1" output
+			(at 135.89 92.71 180)
+			(effects
+				(font
+					(size 1.27 1.27)
+				)
+				(justify left)
+			)
+		)
+		(pin "STBY" output
+			(at 135.89 90.17 180)
+			(effects
+				(font
+					(size 1.27 1.27)
+				)
+				(justify left)
+			)
+		)
