File: Training File/Can.kicad_sch (KiCad schematic)
At the start: 7 parts, among them U2 OKI

Commit message: CAN reciever
Parts:
- removed C1, C2: 10u, symbol Device:C
- removed D1, D2: GRN, symbol Device:LED
- removed R1: 2.2 k, symbol Device:R_US
- removed R2: 820 R, symbol Device:R_US
- removed U2: OKI, symbol MRDT_Devices:OKI
- added C4, C5: 100n, symbol Device:C
- added Conn1: Molex_SL_02, symbol MRDT_Connectors:Molex_SL_02
- added R3: 120, symbol Device:R_US
- added U3: ATA6561-GBQW-N, VDFN8_3X3_MCH, symbol 2026_training_lib:ATA6561-GBQW-N
Connections:
- net +5V: now also C4.1, U3.3 (VCC)
- net GND: now also C4.2, C5.2, U3.2 (GND), U3.9 (EPAD)
- new net: Conn1.1, R3.1, U3.7 (CANH)
- new net: Conn1.2, R3.2, U3.6 (CANL)
- new net +3.3V: C5.1, U3.5 (VIO)
- new net RXD: U3.4 (RXD)
- new net STBY: U3.8 (STBY)
- new net TXD: U3.1 (TXD)

Commit message: Finish schematic
Connections:
- net +3.3V renamed +3V3
Changed lines of the file:
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@@
 	(wire
 		(pts
-			(xy 191.77 97.79) (xy 198.12 97.79)
+			(xy 191.77 97.79) (xy 199.39 97.79)
 		)
 		(stroke
@@
 	)
 	(symbol
+		(lib_id "power:+3V3")
+		(at 199.39 97.79 0)
+		(unit 1)
+		(exclude_from_sim no)
+		(in_bom yes)
+		(on_board yes)
+		(dnp no)
+		(fields_autoplaced yes)
+		(property "Reference" "#PWR014"
+			(at 199.39 101.6 0)
+			(effects
+				(font
+					(size 1.27 1.27)
+				)
+				(hide yes)
+			)
+		)
+		(property "Value" "+3V3"
+			(at 199.39 92.71 0)
+			(effects
+				(font
+					(size 1.27 1.27)
+				)
+			)
+		)
+		(property "Footprint" ""
+			(at 199.39 97.79 0)
+			(effects
+				(font
+					(size 1.27 1.27)
+				)
+				(hide yes)
+			)
+		)
+		(property "Datasheet" ""
+			(at 199.39 97.79 0)
+			(effects
+				(font
+					(size 1.27 1.27)
+				)
+				(hide yes)
+			)
+		)
+		(property "Description" "Power symbol creates a global label with name \"+3V3\""
+			(at 199.39 97.79 0)
+			(effects
+				(font
+					(size 1.27 1.27)
+				)
+				(hide yes)
+			)
+		)
+		(pin "1"
+		)
+		(instances
+			(project ""
+				(path "/d3b46590-8d43-4cdb-9712-6960f55d7470/e486201a-d804-40b0-98ee-00f98b92e5dd"
+					(reference "#PWR014")
+					(unit 1)
+				)
+			)
+		)
+	)
+	(symbol
 		(lib_id "power:+5V")
 		(at 115.57 102.87 0)
@@
 					(unit 1)
 				)
-			)
-		)
-	)
-	(symbol
-		(lib_id "power:+3.3V")
-		(at 198.12 97.79 0)
-		(unit 1)
-		(exclude_from_sim no)
-		(in_bom yes)
-		(on_board yes)
-		(dnp no)
-		(fields_autoplaced yes)
-		(property "Reference" "#PWR014"
-			(at 198.12 101.6 0)
-			(effects
-				(font
-					(size 1.27 1.27)
-				)
-				(hide yes)
-			)
-		)
-		(property "Value" "+3.3V"
-			(at 198.12 92.71 0)
-			(effects
-				(font
-					(size 1.27 1.27)
-				)
-			)
-		)
-		(property "Footprint" ""
-			(at 198.12 97.79 0)
-			(effects
-				(font
-					(size 1.27 1.27)
-				)
-				(hide yes)
-			)
-		)
-		(property "Datasheet" ""
-			(at 198.12 97.79 0)
-			(effects
-				(font
-					(size 1.27 1.27)
-				)
-				(hide yes)
-			)
-		)
-		(property "Description" "Power symbol creates a global label with name \"+3.3V\""
-			(at 198.12 97.79 0)
-			(effects
-				(font
-					(size 1.27 1.27)
-				)
-				(hide yes)
-			)
-		)
-		(pin "1"
-		)
-		(instances
-			(project ""
-				(path "/d3b46590-8d43-4cdb-9712-6960f55d7470/e486201a-d804-40b0-98ee-00f98b92e5dd"
-					(reference "#PWR014")
-					(unit 1)
-				)
