File: TrainingStuff/MCU.kicad_sch (KiCad schematic)
At the start: 0 parts

Commit message: Add Ethernet
Parts:
- added C3: 0.1u, symbol Device:C
- added J1: RJ45_LED_Shielded, symbol Connector:RJ45_LED_Shielded
- added U2: Teensy4.1_DEV-16771, MODULE_DEV-16771, symbol MRDT_Shields:Teensy4.1_DEV-16771
Connections:
- new net: C3.1, J1.2, J1.5
- new net: U2.3.3V_1 (3.3V), U2.3.3V_2 (3.3V), U2.3.3V_3 (3.3V)
- new net: U2.USB_GND1 (USB_GND), U2.USB_GND2 (USB_GND)
- new net +5V: U2.5V
- new net GND: C3.2, J1.8, J1.9, J1.SH, U2.GND1 (GND), U2.GND2 (GND), U2.GND3 (GND), U2.GND4 (GND), U2.GND5 (GND)
- new net LED: J1.10, U2.LED
- new net Rx+: J1.4, U2.R+
- new net Rx-: J1.6, U2.R-
- new net Tx+: J1.1, U2.T+
- new net Tx-: J1.3, U2.T-
- no-connect marks 0 -> 8

Commit message: Add Schematic
Connections:
- net STBY: now reaches U2.2 (OUT2)
- net CTX1: now reaches U2.22 (A8)
- net CRX1: now reaches U2.23 (A9)
- net +3V3: now reaches U2.3.3V_1 (3.3V), U2.3.3V_2 (3.3V), U2.3.3V_3 (3.3V)
- no-connect marks 8 -> 7
Changed lines of the file:
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@@
-	)
-	(no_connect
-		(at 127 50.8)
 	)
 	(no_connect
@@
 	(wire
 		(pts
+			(xy 127 137.16) (xy 134.62 137.16)
+		)
+		(stroke
+			(width 0)
+			(type default)
+		)
+	)
+	(wire
+		(pts
 			(xy 163.83 69.85) (xy 163.83 74.93)
 		)
@@
 	(wire
 		(pts
+			(xy 127 83.82) (xy 133.35 83.82)
+		)
+		(stroke
+			(width 0)
+			(type default)
+		)
+	)
+	(wire
+		(pts
+			(xy 127 50.8) (xy 135.89 50.8)
+		)
+		(stroke
+			(width 0)
+			(type default)
+		)
+	)
+	(wire
+		(pts
 			(xy 166.37 69.85) (xy 166.37 74.93)
 		)
@@
 	(wire
 		(pts
+			(xy 72.39 137.16) (xy 86.36 137.16)
+		)
+		(stroke
+			(width 0)
+			(type default)
+		)
+	)
+	(wire
+		(pts
 			(xy 176.53 69.85) (xy 176.53 88.9)
 		)
@@
 		(pts
 			(xy 127 60.96) (xy 134.62 60.96)
+		)
+		(stroke
+			(width 0)
+			(type default)
+		)
+	)
+	(wire
+		(pts
+			(xy 135.89 39.37) (xy 135.89 50.8)
 		)
 		(stroke
@@
 		)
 	)
+	(hierarchical_label "CTX1"
+		(shape output)
+		(at 72.39 137.16 180)
+		(effects
+			(font
+				(size 1.27 1.27)
+			)
+			(justify right)
+		)
+	)
 	(hierarchical_label "Tx+"
 		(shape input)
@@
 		)
 	)
+	(hierarchical_label "CRX1"
+		(shape input)
+		(at 134.62 137.16 0)
+		(effects
+			(font
+				(size 1.27 1.27)
+			)
+			(justify left)
+		)
+	)
 	(hierarchical_label "Rx-"
 		(shape input)
@@
 		(shape input)
 		(at 134.62 60.96 0)
+		(effects
+			(font
+				(size 1.27 1.27)
+			)
+			(justify left)
+		)
+	)
+	(hierarchical_label "STBY"
+		(shape output)
+		(at 133.35 83.82 0)
 		(effects
 			(font
@@
 					(unit 1)
 				)
+			)
+		)
+	)
+	(symbol
+		(lib_id "power:+3V3")
+		(at 135.89 39.37 0)
+		(unit 1)
+		(exclude_from_sim no)
+		(in_bom yes)
+		(on_board yes)
+		(dnp no)
+		(fields_autoplaced yes)
+		(property "Reference" "#PWR016"
+			(at 135.89 43.18 0)
+			(effects
+				(font
+					(size 1.27 1.27)
+				)
+				(hide yes)
+			)
+		)
+		(property "Value" "+3V3"
+			(at 135.89 34.29 0)
+			(effects
+				(font
+					(size 1.27 1.27)
+				)
+			)
+		)
+		(property "Footprint" ""
+			(at 135.89 39.37 0)
+			(effects
+				(font
+					(size 1.27 1.27)
+				)
+				(hide yes)
+			)
+		)
+		(property "Datasheet" ""
+			(at 135.89 39.37 0)
+			(effects
+				(font
+					(size 1.27 1.27)
+				)
+				(hide yes)
+			)
+		)
+		(property "Description" "Power symbol creates a global label with name \"+3V3\""
+			(at 135.89 39.37 0)
+			(effects
+				(font
+					(size 1.27 1.27)
+				)
+				(hide yes)
+			)
+		)
+		(pin "1"
+		)
+		(instances
+			(project ""
+				(path "/7bedb2c1-4b41-4164-a76e-e6479fce2d5a/4414a215-c08b-405b-96fa-ed5b77b45b9e"
+					(reference "#PWR016")
+					(unit 1)
+				)
